File: ruetueta-pcb.kicad_sch (KiCad schematic)
At the start: 32 parts, among them J1 Conn_01x02, Q1 BC557, Q2 BC557, Q3 BC557, Q4 BC557, Q5 BC557

Commit message: changed footprint for and placement of transistors; moved most components and vias away from ruetueta logo
Parts:
- Q1, Q2, Q3, Q4, Q5: footprint Package_TO_SOT_THT:TO-92_Inline -> Package_TO_SOT_THT:TO-92L_Inline_Wide
Changed lines of the file:
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@@
       (effects (font (size 1.27 1.27)) (justify left))
     )
-    (property "Footprint" "Package_TO_SOT_THT:TO-92_Inline" (id 2) (at 91.44 45.085 0)
+    (property "Footprint" "Package_TO_SOT_THT:TO-92L_Inline_Wide" (id 2) (at 91.44 45.085 0)
       (effects (font (size 1.27 1.27) italic) (justify left) hide)
     )
@@
       (effects (font (size 1.27 1.27)) (justify left))
     )
-    (property "Footprint" "Package_TO_SOT_THT:TO-92_Inline" (id 2) (at 54.61 37.465 0)
+    (property "Footprint" "Package_TO_SOT_THT:TO-92L_Inline_Wide" (id 2) (at 54.61 37.465 0)
       (effects (font (size 1.27 1.27) italic) (justify left) hide)
     )
@@
       (effects (font (size 1.27 1.27)) (justify left))
     )
-    (property "Footprint" "Package_TO_SOT_THT:TO-92_Inline" (id 2) (at 128.27 52.705 0)
+    (property "Footprint" "Package_TO_SOT_THT:TO-92L_Inline_Wide" (id 2) (at 128.27 52.705 0)
       (effects (font (size 1.27 1.27) italic) (justify left) hide)
     )
@@
       (effects (font (size 1.27 1.27)) (justify left))
     )
-    (property "Footprint" "Package_TO_SOT_THT:TO-92_Inline" (id 2) (at 165.1 60.325 0)
+    (property "Footprint" "Package_TO_SOT_THT:TO-92L_Inline_Wide" (id 2) (at 165.1 60.325 0)
       (effects (font (size 1.27 1.27) italic) (justify left) hide)
     )
@@
       (effects (font (size 1.27 1.27)) (justify left))
     )
-    (property "Footprint" "Package_TO_SOT_THT:TO-92_Inline" (id 2) (at 201.93 67.945 0)
+    (property "Footprint" "Package_TO_SOT_THT:TO-92L_Inline_Wide" (id 2) (at 201.93 67.945 0)
       (effects (font (size 1.27 1.27) italic) (justify left) hide)
     )
@@
     )
     (path "/527346bb-ea73-4a6b-90c5-e15d8df2e57f"
-      (reference "Q1") (unit 1) (value "BC557") (footprint "Package_TO_SOT_THT:TO-92_Inline")
+      (reference "Q1") (unit 1) (value "BC557") (footprint "Package_TO_SOT_THT:TO-92L_Inline_Wide")
     )
     (path "/338b4002-dc3b-4d3b-9469-06af0468e64e"
-      (reference "Q2") (unit 1) (value "BC557") (footprint "Package_TO_SOT_THT:TO-92_Inline")
+      (reference "Q2") (unit 1) (value "BC557") (footprint "Package_TO_SOT_THT:TO-92L_Inline_Wide")
     )
     (path "/7e7e285d-7f65-4d53-b55d-ef8b716b04ad"
-      (reference "Q3") (unit 1) (value "BC557") (footprint "Package_TO_SOT_THT:TO-92_Inline")
+      (reference "Q3") (unit 1) (value "BC557") (footprint "Package_TO_SOT_THT:TO-92L_Inline_Wide")
     )
     (path "/94111311-3b6f-42c7-9d02-059d31ce3d9b"
-      (reference "Q4") (unit 1) (value "BC557") (footprint "Package_TO_SOT_THT:TO-92_Inline")
+      (reference "Q4") (unit 1) (value "BC557") (footprint "Package_TO_SOT_THT:TO-92L_Inline_Wide")
     )
     (path "/b17aeaab-26ca-44cd-bb3c-91ac53a5dbe1"
-      (reference "Q5") (unit 1) (value "BC557") (footprint "Package_TO_SOT_THT:TO-92_Inline")
+      (reference "Q5") (unit 1) (value "BC557") (footprint "Package_TO_SOT_THT:TO-92L_Inline_Wide")
     )
     (path "/f377b136-56b5-4e23-8cd2-f732b5942e28"
